File: LPC1768.sch (EAGLE design)
At the start: 84 parts, among them CON1 USB-MB-S, CON2 USB-MB-S, CON3 RJ45, CON4 USB-A-H, IC1 LD1117S33, IC3 LD1117S33, IC4 LPC1768, IC5 DP83848J, Q2 32.768kHz, Q3 12MHz, Q4 12MHz, SW1 SPST, SW2 SPST, T1 BSS84, T2 BSS84

Commit message: Added mbed HDK library. Modified schematic and added board. Added BOM. Added some drc files.
Parts:
- removed C25, C29: 10uF, mbed-HDK:C-POLB
- removed C26, C27, C28, C30, C31, C32, C33, C34, C35, C36, C37: 100nF, mbed-HDK:C0603
- removed CON3: RJ45, mbed-HDK:RJ45
- removed CON4: USB-A-H, mbed-HDK:USB-A-H
- removed IC5: DP83848J, mbed-HDK:DP83848J
- removed OSC1: 50MHz, mbed-HDK:OSCILLATOR
- removed Q3, Q4: 12MHz, mbed-HDK:Q_HC49UP
- removed R14: 4k87, mbed-HDK:R0603
- removed R15, R17, R18, R19: 49R9, mbed-HDK:R0603
- removed R16: 2k2, mbed-HDK:R0603
- removed R22, R23: 15k, mbed-HDK:R0603
- added SV1, SV3: (no value), con-lstb:MA06-1
- added SV2: (no value), con-lstb:MA06-2
- added SV4: (no value), con-lstb:MA03-2
- added SV5: (no value), con-lstb:MA08-1
- added SV6, SV7: (no value), con-lstb:MA04-1
- added X1, X2: 12MHz, crystals_oscillators:ABM8
- C23, C24, C8, C9: value 18pF -> 27pF
Connections:
- removed net CON2: CON3.6, IC5.RD-, R19.P$1
- removed net N$10: C11.P$1, D1.K, D2.K, IC3.IN
- removed net N$123: IC5.RBIAS, R14.P$2
- removed net N$127: IC5.RX_DV/MII_MODE, R16.P$2
- removed net N$22: C24.P$2, IC4.X2, Q3.2
- removed net PFBOUT: C28.P$2, C29.1, C30.P$2, C34.P$1, IC5.PFBIN1, IC5.PFBIN2, IC5.PFBOUT
- removed net RD+: CON3.4, IC5.RD+, R18.P$2
- removed net TD+: CON3.1, IC5.TD+, R15.P$2
- removed net TD-: CON3.3, IC5.TD-, R17.P$1
- removed net VBAT: IC4.VBAT
- new net N$27: IC4.P1.18/USB_UP/PWM1.1/CAP1.0
- new net N$30: IC4.P1.19/MC0A/USB_PPWR/CAP1.1
- new net N$31: IC4.P1.20/MCFB0/PWM1.2/SCK0
- new net N$32: IC4.P1.21/MCABORT/PWM1.3/SSEL0
- new net N$33: IC4.P1.22/MC0B/USB_PWRD/MAT1.0
- new net N$34: IC4.P1.23/MCFB1/PWM1.4/MISO0
- new net N$35: IC4.P1.24/MCFB2/PWM1.5/MOSI0
- new net N$36: IC4.P1.29/MC2B/PCAP1.1/MAT0.1
- new net N$37: IC4.P1.30/VBUS/AD0.4
- new net N$38: IC4.P1.31/SCK1/AD0.5
- new net N$39: IC4.P2.0/PWM1.1/TXD1/TRACECLK, SV5.8
- new net N$40: IC4.P2.1/PWM1.2/RXD1, SV5.7
- new net N$41: IC4.P2.2/PWM1.3/CTS1/TRACEDATA3, SV5.6
- new net N$42: IC4.P2.3/PWM1.4/DCD1/TRACEDATA2, SV5.5
- new net N$43: IC4.P2.4/PWM1.5/DSR1/TRACEDATA1, SV5.4
- new net N$44: IC4.P2.5/PWM1.6/DTR1/TRACEDATA0, SV5.3
- new net N$45: IC4.P2.6/PCAP1.0/RI1/TRACECLK, SV5.2
- new net N$46: IC4.P2.7/CAN_RX2/RTS1, SV5.1
- new net N$47: IC4.P2.8/CAN_TX2/TXD2
- new net N$48: IC4.P2.11/EINT1N/I2STX_CLK
- new net N$49: IC4.P2.12/EINT2N/I2STX_WS
- new net N$50: IC4.P2.13/EINT3N/I2STX_SDA
- new net N$51: IC4.P3.25/MAT0.0/PWM1.2
- new net N$52: IC4.P3.26/STCLK/MAT0.1/PWM1.3
- new net N$53: IC4.P4.28/RX_MCLK/MAT2.0/TXD3
- new net N$54: IC4.P4.29/TX_MCLK/MAT2.1/RXD3
- new net N$55: IC4.P0.28/SCL0/USB_SCL
- new net N$56: IC4.P0.27/SDA0/USB_SDA
- new net N$57: IC4.P0.26/AD0.3/AOUT/RXD3
- new net N$58: IC4.P0.25/AD0.2/I2SRX_SDA/TXD3
- new net N$59: IC4.P0.24/AD0.1/I2SRX_WS/CAP3.1
- new net N$60: IC4.P0.23/AD0.0/I2SRX_CLK/CAP3.0
- new net N$61: IC4.P0.22/RTS1/CAN_TX1
- new net N$62: IC4.P0.21/RI1/CAN_RX1
- new net N$63: IC4.P0.20/DTR1/SCL1
- new net N$64: IC4.P0.19/DSR1/MCICLK/SDA1
- new net N$65: IC4.P0.18/DCD1/MOSI0/MOSI1
- new net N$66: IC4.P0.17/CTS1/MISO0/MISO
- new net N$67: IC4.P0.16/RXD1/SSEL0/SSEL
- new net N$68: IC4.P0.11/RXD2/SCL2/MAT3.1
- new net N$69: IC4.P0.10/TXD2/SDA2/MAT3.0
- new net N$70: IC4.P0.9/I2STX_SDA/MOSI1/MAT2.3
- new net N$71: IC4.P0.8/I2STX_WS/MISO1/MAT2.2
- new net N$72: IC4.P0.7/I2STX_CLK/SCK1/MAT2.1
- new net N$73: IC4.P0.6/I2SRX_SDA/SSEL1/MAT2.0
- new net N$74: IC4.P0.5/I2SRX_WS/CAN_TX2/CAP2.1
- new net N$75: IC4.P0.4/I2SRX_CLK/CAN_RX2/CAP2.0
- new net N$76: IC4.P0.1/CAN_TX1/RXD3/SCL1
- new net N$77: IC4.P0.0/CAN_RX1/TXD3/SDA1
- new net N$78: C24.P$2, IC4.X2, X2.X2
- new net N$79: IC2.NC11, SV1.6
- new net N$80: IC2.NC10, SV1.5
- new net N$81: IC2.SLEEP_NREQ, SV1.4
- new net N$82: IC2.WAKE_NREQ, SV1.3
- new net N$83: IC2.NC9, SV1.2
- new net N$84: IC2.NC8, SV1.1
- new net N$85: IC2.NC2, SV3.6
- new net N$86: IC2.NC3, SV3.5
- new net N$87: IC2.NC4, SV3.4
- new net N$88: IC2.NC5, SV3.3
- new net N$89: IC2.NC6, SV3.2
- new net N$90: IC2.NC7, SV3.1
- new net TGT_NRESET1: IC2.TGT_NRESET, SV2.6
- new net TGT_RX1: IC2.TGT_RX, SV2.2
- new net TGT_SWCLK1: IC2.TGT_SWCLK, SV2.12
- new net TGT_SWDIO1: IC2.TGT_SWDIO, SV2.10
- new net TGT_SWO1: IC2.TGT_SWO, SV2.8
- new net TGT_TX1: IC2.TGT_TX, SV2.4
- new net VBUS_MIX: C11.P$1, D1.K, D2.K, IC3.IN, SV4.3, SV4.4
- net +3.3V_TGT: now also SV4.5, SV4.6; no longer C25.1, C26.P$1, C27.P$1, C31.P$1, C32.P$1, C33.P$1, C35.P$1, C36.P$2, C37.P$2, CON3.2, CON3.5, IC5.AVDD33, IC5.IOVDD33@1, IC5.IOVDD33@2, OSC1.VCC, R15.P$1, R16.P$1, R17.P$2, R18.P$1, R19.P$2
- net 50MHZ: now also SV7.1; no longer IC5.X1, OSC1.CLK
- net ETH_OSC_EN: no longer OSC1.EN
- net ETH_RST: no longer IC5.RESET_N
- net GND: now also SV4.1, SV4.2, X1.GND@1, X1.GND@2, X2.GND@1, X2.GND@2; no longer C25.2, C26.P$2, C27.P$2, C28.P$1, C29.2, C30.P$1, C31.P$2, C32.P$2, C33.P$2, C34.P$2, C35.P$2, C36.P$1, C37.P$1, CON3.SHIELD1, CON3.SHIELD2, CON4.GND, IC5.AGND@1, IC5.AGND@2, IC5.DGND, IC5.GNDPAD, IC5.IOGND@2, OSC1.GND, R14.P$1, R22.P$1, R23.P$1
- net LED_LINK: no longer IC5.LED_LINK/AN0
- net LED_SPEED: no longer IC5.LED_SPEED/AN1
- net N$11: now also X1.X1; no longer Q4.1
- net N$12: now also X1.X2; no longer Q4.2
- net N$21: now also X2.X1; no longer Q3.1
- net TGT_D+: no longer CON4.D+, R22.P$2
- net TGT_D-: no longer CON4.D-, R23.P$2
- net TGT_NRESET: now also SV2.5; no longer IC2.TGT_NRESET
- net TGT_P1.0: now also SV6.4; no longer IC5.TXD_0
- net TGT_P1.1: now also SV6.3; no longer IC5.TXD_1
- net TGT_P1.10: now also SV7.3; no longer IC5.RXD_1/PHYAD2
- net TGT_P1.14: now also SV7.2; no longer IC5.RX_ER/MDIX_EN
- net TGT_P1.16: no longer IC5.MDC
- net TGT_P1.17: no longer IC5.MDIO
- net TGT_P1.4: now also SV6.2; no longer IC5.TX_EN
- net TGT_P1.8: now also SV6.1; no longer IC5.CRS/CRS_DV/LED_CFG
- net TGT_P1.9: now also SV7.4; no longer IC5.RXD_0/PHYAD1
- net TGT_RX: now also SV2.1; no longer IC2.TGT_RX
- net TGT_SWCLK: now also SV2.11; no longer IC2.TGT_SWCLK
- net TGT_SWDIO: now also SV2.9; no longer IC2.TGT_SWDIO
- net TGT_SWO: now also SV2.7
- net TGT_TX: now also SV2.3; no longer IC2.TGT_TX
- net VBUS_IF: no longer CON4.VBUS
Other:
- note removed: "Decoupling cap close to OSC2"
- note removed: "Route with matched signal traces"
- moved on the sheet: C21, C22, C23, C24, C8, C9, Q2
